File: ucpd-passthrough.kicad_pcb (KiCad board)
At the start: 2 copper layers, 50 x 50 mm, 60 parts, among them J1 Output, J2 USB Data passthrough, J3 UART, J4 Display, J5 SWD, J6 USB MCU, J7 VIN, J8 VOUT, Q1 2N7002, U1 STM32G0B1CETxN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

Commit message: Update pcb values from schematic
Parts:
- removed REF**: OSHW-Symbol_6.7x6mm_SilkScreen, Symbol:OSHW-Symbol_6.7x6mm_SilkScreen
- R10, R11, R12, R18: value 1K -> 100
- R16, R3: value 10k -> 10K
- R9: value 1K -> 220
