File: mcu.kicad_sch (KiCad schematic)
At the start: 20 parts, among them J3 UART, J4 Display, J5 SWD, U1 STM32G0B1CETxN, U2 MIC5504-3.3YM5

Commit message: Clarify licenses
Other:
- title: (none) -> UCPD-Passthrough
Changed lines of the file:
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@@
 	(generator_version "8.0")
 	(paper "A4")
+	(title_block
+		(title "UCPD-Passthrough")
+		(rev "0.1")
+		(comment 1 "License: CERN-OHL-P-2.0")
+	)
 	(junction
 		(at 143.51 38.1)
