File: pd.kicad_sch (KiCad schematic)
At the start: 12 parts

Commit message: Clarify licenses
Other:
- title: (none) -> UCPD-Passthrough
Changed lines of the file:
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@@
 	(generator_version "8.0")
 	(paper "A4")
+	(title_block
+		(title "UCPD-Passthrough")
+		(rev "0.1")
+		(comment 1 "License: CERN-OHL-P-2.0")
+	)
 	(junction
 		(at 118.11 87.63)
